File: examples/OLINUXINO/A10-A20-OLINUXINO-MICRO-4GB_Rev_D/kicad_files/A10-A20-OLINUXINO-MICRO-4GB_Rev_D.kicad_pcb (KiCad board)
At the start: 4 copper layers, 142.2 x 82.6 mm, 558 parts, among them Q1 4SB25.000F20E15/5x3.2mm/20ppm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, Q2 32768Hz/6pF, Q3 4SB24.000F20E15/5x3.2mm/20ppm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, T1 BC846B, U1 A10/A20, U10 SY6280, U11 SY6280, U12 AXP209(QFN48), U13 SY8008C(AA)C, U14 MP1482DS, U15 SY8008C(AA)C, U16 SY7208(SOT23-6), U17 RCLAMP0524P, U2 H5TQ2G63BFR_MEM4G16D3EABG-125, U22 RCLAMP0524P, U23 RCLAMP0524P, U3 H5TQ2G63BFR_MEM4G16D3EABG-125, U6 AT24C16BN-SH, U7 RTL8201CP, U8 H27UBG8T2BTR, U9 SY6280

Commit message: replace / in deice name with _, to Fix few problems
Parts:
- 5V_E_SATA233: value ~ -> (none)
Connections:
- net /+15V renamed +15V
- net /+24V renamed +24V
- net /+5V renamed +5V
- net /+5V_OTG_PWR renamed +5V_OTG_PWR
- net /ADBG renamed ADBG
- net /BA0 renamed BA0
- net /BA1 renamed BA1
- net /BA2 renamed BA2
- net /CASN renamed CASN
- net /CKE renamed CKE
- net /CLK renamed CLK
- net /CLKN renamed CLKN
- net /CPU-REF renamed CPU-REF
- net /DDR3_ODT renamed DDR3_ODT
- net /DDR3_RST renamed DDR3_RST
- net /DDR3_SA0 renamed DDR3_SA0
- net /DDR3_SA1 renamed DDR3_SA1
- net /DDR3_SA10 renamed DDR3_SA10
- net /DDR3_SA11 renamed DDR3_SA11
- net /DDR3_SA12 renamed DDR3_SA12
- net /DDR3_SA13 renamed DDR3_SA13
- net /DDR3_SA14 renamed DDR3_SA14
- net /DDR3_SA15 renamed DDR3_SA15
- net /DDR3_SA2 renamed DDR3_SA2
- net /DDR3_SA3 renamed DDR3_SA3
- net /DDR3_SA4 renamed DDR3_SA4
- net /DDR3_SA5 renamed DDR3_SA5
- net /DDR3_SA6 renamed DDR3_SA6
- net /DDR3_SA7 renamed DDR3_SA7
- net /DDR3_SA8 renamed DDR3_SA8
- net /DDR3_SA9 renamed DDR3_SA9
- net /DDR3_SBA0 renamed DDR3_SBA0
- net /DDR3_SBA1 renamed DDR3_SBA1
- net /DDR3_SBA2 renamed DDR3_SBA2
- net /DDR3_SCAS renamed DDR3_SCAS
- net /DDR3_SCS0 renamed DDR3_SCS0
- net /DDR3_SDQM0 renamed DDR3_SDQM0
- net /DDR3_SDQM1 renamed DDR3_SDQM1
- net /DDR3_SDQM2 renamed DDR3_SDQM2
- net /DDR3_SDQM3 renamed DDR3_SDQM3
- net /DDR3_SDQS0 renamed DDR3_SDQS0
- net /DDR3_SDQS0# renamed DDR3_SDQS0#
- net /DDR3_SDQS1 renamed DDR3_SDQS1
- net /DDR3_SDQS1# renamed DDR3_SDQS1#
- net /DDR3_SDQS2 renamed DDR3_SDQS2
- net /DDR3_SDQS2# renamed DDR3_SDQS2#
- net /DDR3_SDQS3 renamed DDR3_SDQS3
- net /DDR3_SDQS3# renamed DDR3_SDQS3#
- net /DDR3_SRAS renamed DDR3_SRAS
- net /DDR3_SWE renamed DDR3_SWE
- net /DDR_VREF renamed DDR_VREF
- net /DQ0 renamed DQ0
- net /DQ1 renamed DQ1
- net /DQ10 renamed DQ10
- net /DQ11 renamed DQ11
- net /DQ12 renamed DQ12
- net /DQ13 renamed DQ13
- net /DQ14 renamed DQ14
- net /DQ15 renamed DQ15
- net /DQ16 renamed DQ16
- net /DQ17 renamed DQ17
- net /DQ18 renamed DQ18
- net /DQ19 renamed DQ19
- net /DQ2 renamed DQ2
- net /DQ20 renamed DQ20
- net /DQ21 renamed DQ21
- net /DQ22 renamed DQ22
- net /DQ23 renamed DQ23
- net /DQ24 renamed DQ24
- net /DQ25 renamed DQ25
- net /DQ26 renamed DQ26
- net /DQ27 renamed DQ27
- net /DQ28 renamed DQ28
- net /DQ29 renamed DQ29
- net /DQ3 renamed DQ3
- net /DQ30 renamed DQ30
- net /DQ31 renamed DQ31
- net /DQ4 renamed DQ4
- net /DQ5 renamed DQ5
- net /DQ6 renamed DQ6
- net /DQ7 renamed DQ7
- net /DQ8 renamed DQ8
- net /DQ9 renamed DQ9
- net /ECOL renamed ECOL
- net /ECRS renamed ECRS
- net /EMDC renamed EMDC
- net /EMDIO renamed EMDIO
- net /ENTER_BUT renamed ENTER_BUT
- net /EPHY-RST# renamed EPHY-RST#
- net /ERXCK renamed ERXCK
- net /ERXD0 renamed ERXD0
- net /ERXD1 renamed ERXD1
- net /ERXD2 renamed ERXD2
- net /ERXD3 renamed ERXD3
- net /ERXDV renamed ERXDV
- net /ERXERR renamed ERXERR
- net /ESC_BUT renamed ESC_BUT
- net /ETXCK renamed ETXCK
- net /ETXD0 renamed ETXD0
- net /ETXD1 renamed ETXD1
- net /ETXD2 renamed ETXD2
- net /ETXD3 renamed ETXD3
- net /ETXEN renamed ETXEN
- net /EXTEN renamed EXTEN
- net /FMINL renamed FMINL
- net /FMINR renamed FMINR
- net /GNDA renamed GNDA
- net /GPIO1 renamed GPIO1
- net /GPIO2 renamed GPIO2
- net /GPIO3 renamed GPIO3
- net /HCEC renamed HCEC
- net /HDMI_5V_SOURCE renamed HDMI_5V_SOURCE
- net /HHPD renamed HHPD
- net /HOME_BUT renamed HOME_BUT
- net /HPCOM renamed HPCOM
- net /HPOUTL renamed HPOUTL
- net /HPOUTR renamed HPOUTR
- net /HSCL renamed HSCL
- net /HSDA renamed HSDA
- net /HTX0N renamed HTX0N
- net /HTX0P renamed HTX0P
- net /HTX1N renamed HTX1N
- net /HTX1P renamed HTX1P
- net /HTX2N renamed HTX2N
- net /HTX2P renamed HTX2P
- net /HTXCN renamed HTXCN
- net /HTXCP renamed HTXCP
- net /IPSOUT renamed IPSOUT
- net /LCD_CLK renamed LCD_CLK
- net /LCD_D0 renamed LCD_D0
- net /LCD_D1 renamed LCD_D1
- net /LCD_D10 renamed LCD_D10
- net /LCD_D11 renamed LCD_D11
- net /LCD_D12 renamed LCD_D12
- net /LCD_D13 renamed LCD_D13
- net /LCD_D14 renamed LCD_D14
- net /LCD_D15 renamed LCD_D15
- net /LCD_D16 renamed LCD_D16
- net /LCD_D17 renamed LCD_D17
- net /LCD_D18 renamed LCD_D18
- net /LCD_D19 renamed LCD_D19
- net /LCD_D2 renamed LCD_D2
- net /LCD_D20 renamed LCD_D20
- net /LCD_D21 renamed LCD_D21
- net /LCD_D22 renamed LCD_D22
- net /LCD_D23 renamed LCD_D23
- net /LCD_D3 renamed LCD_D3
- net /LCD_D4 renamed LCD_D4
- net /LCD_D5 renamed LCD_D5
- net /LCD_D6 renamed LCD_D6
- net /LCD_D7 renamed LCD_D7
- net /LCD_D8 renamed LCD_D8
- net /LCD_D9 renamed LCD_D9
- net /LCD_DE renamed LCD_DE
- net /LCD_HSYNC renamed LCD_HSYNC
- net /LCD_PWR renamed LCD_PWR
- net /LCD_VSYNC renamed LCD_VSYNC
- net /LDO3_2.8V renamed LDO3_2.8V
- net /LDO4_2.8V renamed LDO4_2.8V
- net /LINEINL renamed LINEINL
- net /LINEINR renamed LINEINR
- net /LRADC0 renamed LRADC0
- net /LRADC1 renamed LRADC1
- net /MENU_BUT renamed MENU_BUT
- net /MIC1OUTN renamed MIC1OUTN
- net /MIC1OUTP renamed MIC1OUTP
- net /MICIN1 renamed MICIN1
- net /MICIN2 renamed MICIN2
- net /MICM renamed MICM
- net /N$1 renamed N$1
- net /N$10 renamed N$10
- net /N$100 renamed N$100
- net /N$101 renamed N$101
- net /N$102 renamed N$102
- net /N$105 renamed N$105
- net /N$106 renamed N$106
- net /N$11 renamed N$11
- net /N$111 renamed N$111
- net /N$112 renamed N$112
- net /N$113 renamed N$113
- net /N$114 renamed N$114
- net /N$115 renamed N$115
- net /N$116 renamed N$116
- net /N$119 renamed N$119
- net /N$12 renamed N$12
- net /N$120 renamed N$120
- net /N$121 renamed N$121
- net /N$122 renamed N$122
- net /N$123 renamed N$123
- net /N$124 renamed N$124
- net /N$125 renamed N$125
- net /N$126 renamed N$126
- net /N$127 renamed N$127
- net /N$128 renamed N$128
- net /N$129 renamed N$129
- net /N$13 renamed N$13
- net /N$130 renamed N$130
- net /N$131 renamed N$131
- net /N$132 renamed N$132
- net /N$133 renamed N$133
- net /N$134 renamed N$134
- net /N$135 renamed N$135
- net /N$137 renamed N$137
- net /N$139 renamed N$139
- net /N$14 renamed N$14
- net /N$140 renamed N$140
- net /N$15 renamed N$15
- net /N$16 renamed N$16
- net /N$161 renamed N$161
- net /N$17 renamed N$17
- net /N$176 renamed N$176
- net /N$18 renamed N$18
- net /N$187 renamed N$187
- net /N$19 renamed N$19
- net /N$190 renamed N$190
- net /N$191 renamed N$191
- net /N$192 renamed N$192
- net /N$193 renamed N$193
- net /N$194 renamed N$194
- net /N$195 renamed N$195
- net /N$196 renamed N$196
- net /N$197 renamed N$197
- net /N$2 renamed N$2
- net /N$20 renamed N$20
- net /N$21 renamed N$21
- net /N$22 renamed N$22
- net /N$220 renamed N$220
- net /N$221 renamed N$221
- net /N$222 renamed N$222
- net /N$223 renamed N$223
- net /N$229 renamed N$229
- net /N$23 renamed N$23
- net /N$230 renamed N$230
- net /N$231 renamed N$231
- net /N$232 renamed N$232
- net /N$24 renamed N$24
- net /N$25 renamed N$25
- net /N$26 renamed N$26
- net /N$266 renamed N$266
- net /N$27 renamed N$27
- net /N$28 renamed N$28
- net /N$3 renamed N$3
- net /N$31 renamed N$31
- net /N$32 renamed N$32
- net /N$33 renamed N$33
- net /N$34 renamed N$34
- net /N$35 renamed N$35
- net /N$36 renamed N$36
- net /N$37 renamed N$37
- net /N$38 renamed N$38
- net /N$39 renamed N$39
- net /N$4 renamed N$4
- net /N$40 renamed N$40
- net /N$41 renamed N$41
- net /N$42 renamed N$42
- net /N$43 renamed N$43
- net /N$44 renamed N$44
- net /N$45 renamed N$45
- net /N$46 renamed N$46
- net /N$47 renamed N$47
- net /N$49 renamed N$49
- net /N$5 renamed N$5
- net /N$50 renamed N$50
- net /N$51 renamed N$51
- net /N$53 renamed N$53
- net /N$54 renamed N$54
- net /N$55 renamed N$55
- net /N$56 renamed N$56
- net /N$57 renamed N$57
- net /N$6 renamed N$6
- net /N$60 renamed N$60
- net /N$61 renamed N$61
- net /N$62 renamed N$62
- net /N$64 renamed N$64
- net /N$66 renamed N$66
- net /N$67 renamed N$67
- net /N$68 renamed N$68
- net /N$69 renamed N$69
- net /N$7 renamed N$7
- net /N$78 renamed N$78
- net /N$79 renamed N$79
- net /N$8 renamed N$8
- net /N$80 renamed N$80
- net /N$84 renamed N$84
- net /N$85 renamed N$85
- net /N$86 renamed N$86
- net /N$9 renamed N$9
- net /N$99 renamed N$99
- net /NALE renamed NALE
- net /NAND_DQS renamed NAND_DQS
- net /NCE0 renamed NCE0
- net /NCLE renamed NCLE
- net /NDQ0 renamed NDQ0
- net /NDQ1 renamed NDQ1
- net /NDQ2 renamed NDQ2
- net /NDQ3 renamed NDQ3
- net /NDQ4 renamed NDQ4
- net /NDQ5 renamed NDQ5
- net /NDQ6 renamed NDQ6
- net /NDQ7 renamed NDQ7
- net /NMI_N renamed NMI_N
- net /NRB0 renamed NRB0
- net /NRBO/NRB1 renamed NRBO/NRB1
- net /NRE renamed NRE
- net /NWE renamed NWE
- net /ODT0 renamed ODT0
- net /ODT1 renamed ODT1
- net /PB10 renamed PB10
- net /PB11 renamed PB11
- net /PB12 renamed PB12
- net /PB13 renamed PB13
- net /PB14 renamed PB14
- net /PB15 renamed PB15
- net /PB16 renamed PB16
- net /PB17 renamed PB17
- net /PB2/PWM0 renamed PB2/PWM0
- net /PB3 renamed PB3
- net /PB4 renamed PB4
- net /PB5 renamed PB5
- net /PB6 renamed PB6
- net /PB7 renamed PB7
- net /PB8/SATA-PWR-EN renamed PB8/SATA-PWR-EN
- net /PC16 renamed PC16
- net /PC17 renamed PC17
- net /PC18 renamed PC18
- net /PC23 renamed PC23
- net /PC24/NQS renamed PC24/NQS
- net /PC3/NCE1 renamed PC3/NCE1
- net /PC7/NRB1 renamed PC7/NRB1
- net /PE0 renamed PE0
- net /PE1 renamed PE1
- net /PE10 renamed PE10
- net /PE11 renamed PE11
- net /PE2 renamed PE2
- net /PE3 renamed PE3
- net /PE4 renamed PE4
- net /PE5 renamed PE5
- net /PE6 renamed PE6
- net /PE7 renamed PE7
- net /PE8 renamed PE8
- net /PE9 renamed PE9
- net /PG0 renamed PG0
- net /PG1 renamed PG1
- net /PG10 renamed PG10
- net /PG11 renamed PG11
- net /PG2 renamed PG2
- net /PG3 renamed PG3
- net /PG4 renamed PG4
- net /PG5 renamed PG5
- net /PG6 renamed PG6
- net /PG7 renamed PG7
- net /PG8 renamed PG8
- net /PG9 renamed PG9
- net /PH0 renamed PH0
- net /PH10 renamed PH10
- net /PH11/SDC3-DET# renamed PH11/SDC3-DET#
- net /PH12 renamed PH12
- net /PH13 renamed PH13
- net /PH14 renamed PH14
- net /PH15 renamed PH15
- net /PH16 renamed PH16
- net /PH17 renamed PH17
- net /PH18 renamed PH18
- net /PH19 renamed PH19
- net /PH2/LED renamed PH2/LED
- net /PH20 renamed PH20
- net /PH21 renamed PH21
- net /PH22 renamed PH22
- net /PH23 renamed PH23
- net /PH24 renamed PH24
- net /PH25 renamed PH25
- net /PH26 renamed PH26
- net /PH27 renamed PH27
- net /PH7 renamed PH7
- net /PH9 renamed PH9
- net /PI0 renamed PI0
- net /PI1 renamed PI1
- net /PI10 renamed PI10
- net /PI11 renamed PI11
- net /PI14 renamed PI14
- net /PI15 renamed PI15
- net /PI2 renamed PI2
- net /PI3 renamed PI3
- net /RASN renamed RASN
- net /RESET_N renamed RESET_N
- net /SA0 renamed SA0
- net /SA1 renamed SA1
- net /SA10 renamed SA10
- net /SA11 renamed SA11
- net /SA12 renamed SA12
- net /SA13 renamed SA13
- net /SA14 renamed SA14
- net /SA15 renamed SA15
- net /SA2 renamed SA2
- net /SA3 renamed SA3
- net /SA4 renamed SA4
- net /SA5 renamed SA5
- net /SA6 renamed SA6
- net /SA7 renamed SA7
- net /SA8 renamed SA8
- net /SA9 renamed SA9
- net /SATA-RXM renamed SATA-RXM
- net /SATA-RXP renamed SATA-RXP
- net /SATA-TXM renamed SATA-TXM
- net /SATA-TXP renamed SATA-TXP
- net /SCK renamed SCK
- net /SCK# renamed SCK#
- net /SCKE0 renamed SCKE0
- net /SCKE1 renamed SCKE1
- net /SCS0 renamed SCS0
- net /SDBG0 renamed SDBG0
- net /SDBG1 renamed SDBG1
- net /SDC3-CLK renamed SDC3-CLK
- net /SDC3-CMD renamed SDC3-CMD
- net /SDC3-D0 renamed SDC3-D0
- net /SDC3-D1 renamed SDC3-D1
- net /SDC3-D2 renamed SDC3-D2
- net /SDC3-D3 renamed SDC3-D3
- net /SDQ0 renamed SDQ0
- net /SDQ1 renamed SDQ1
- net /SDQ10 renamed SDQ10
- net /SDQ11 renamed SDQ11
- net /SDQ12 renamed SDQ12
- net /SDQ13 renamed SDQ13
- net /SDQ14 renamed SDQ14
- net /SDQ15 renamed SDQ15
- net /SDQ16 renamed SDQ16
- net /SDQ17 renamed SDQ17
- net /SDQ18 renamed SDQ18
- net /SDQ19 renamed SDQ19
- net /SDQ2 renamed SDQ2
- net /SDQ20 renamed SDQ20
- net /SDQ21 renamed SDQ21
- net /SDQ22 renamed SDQ22
- net /SDQ23 renamed SDQ23
- net /SDQ24 renamed SDQ24
- net /SDQ25 renamed SDQ25
- net /SDQ26 renamed SDQ26
- net /SDQ27 renamed SDQ27
- net /SDQ28 renamed SDQ28
- net /SDQ29 renamed SDQ29
- net /SDQ3 renamed SDQ3
- net /SDQ30 renamed SDQ30
- net /SDQ31 renamed SDQ31
- net /SDQ4 renamed SDQ4
- net /SDQ5 renamed SDQ5
- net /SDQ6 renamed SDQ6
- net /SDQ7 renamed SDQ7
- net /SDQ8 renamed SDQ8
- net /SDQ9 renamed SDQ9
- net /SDQM0 renamed SDQM0
- net /SDQM1 renamed SDQM1
- net /SDQM2 renamed SDQM2
- net /SDQM3 renamed SDQM3
- net /SDQS0 renamed SDQS0
- net /SDQS0_N renamed SDQS0_N
- net /SDQS1 renamed SDQS1
- net /SDQS1_N renamed SDQS1_N
- net /SDQS2 renamed SDQS2
- net /SDQS2_N renamed SDQS2_N
- net /SDQS3 renamed SDQS3
- net /SDQS3_N renamed SDQS3_N
- net /SD_VCC1 renamed SD_VCC1
- net /SEARCH_BUT renamed SEARCH_BUT
- net /SPI1-CLK renamed SPI1-CLK
- net /SPI1-CS0 renamed SPI1-CS0
- net /SPI1-MISO renamed SPI1-MISO
- net /SPI1-MOSI renamed SPI1-MOSI
- net /SPI2-CLK renamed SPI2-CLK
- net /SPI2-CS0 renamed SPI2-CS0
- net /SPI2-MISO renamed SPI2-MISO
- net /SPI2-MOSI renamed SPI2-MOSI
- net /SRST renamed SRST
- net /TPX1 renamed TPX1
- net /TPX2 renamed TPX2
- net /TPY1 renamed TPY1
- net /TPY2 renamed TPY2
- net /TSD_CLK renamed TSD_CLK
- net /TSD_CMD renamed TSD_CMD
- net /TSD_D0 renamed TSD_D0
- net /TSD_D1 renamed TSD_D1
- net /TSD_D2 renamed TSD_D2
- net /TSD_D3 renamed TSD_D3
- net /TVIN0 renamed TVIN0
- net /TVIN1 renamed TVIN1
- net /TVIN2 renamed TVIN2
- net /TVIN3 renamed TVIN3
- net /TVOUT3 renamed TVOUT3
- net /TWI0-SCK renamed TWI0-SCK
- net /TWI0-SDA renamed TWI0-SDA
- net /TWI1-SCK renamed TWI1-SCK
- net /TWI1-SDA renamed TWI1-SDA
- net /TWI2-SCK renamed TWI2-SCK
- net /TWI2-SDA renamed TWI2-SDA
- net /UART0-RX renamed UART0-RX
- net /UART0-TX renamed UART0-TX
- net /UART6-RX renamed UART6-RX
- net /UART6-TX renamed UART6-TX
- net /UART7-RX renamed UART7-RX
- net /UART7-TX renamed UART7-TX
- net /UBOOT_SEL renamed UBOOT_SEL
- net /UDM0 renamed UDM0
- net /UDM1 renamed UDM1
- net /UDM2 renamed UDM2
- net /UDP0 renamed UDP0
- net /UDP1 renamed UDP1
- net /UDP2 renamed UDP2
- net /USB0-DRV renamed USB0-DRV
- net /USB0-IDDET renamed USB0-IDDET
- net /USB0-VBUSDET renamed USB0-VBUSDET
- net /USB1-DRV renamed USB1-DRV
- net /USB2-DRV renamed USB2-DRV
- net /VDD renamed VDD
- net /VDD_RTC renamed VDD_RTC
- net /VGA-B renamed VGA-B
- net /VGA-G renamed VGA-G
- net /VGA-R renamed VGA-R
- net /VGA_HSYNC renamed VGA_HSYNC
- net /VGA_VSYNC renamed VGA_VSYNC
- net /VINT renamed VINT
- net /VMIC renamed VMIC
- net /VOL+_BUT renamed VOL+_BUT
- net /VOL-_BUT renamed VOL-_BUT
- net /VPP renamed VPP
- net /WEN renamed WEN
- 1.2V_CPU233 pad 1: /VCC/2 -> VCC/2
- 1.2V_INT233 pad 1: /VCCINT -> VCCINT
- 1.5V233 pad 1: /V+ -> V+
- 3.3V233 pad 1: /VCC -> VCC
- 5V_PWR233 pad 2: /GND -> GND
- 5V_SATA_PWR233 pad 2: /GND -> GND
- C1 pad 1: /V+ -> V+
- C10 pad 1: /GND -> GND
- C10 pad 2: /V+ -> V+
- C100 pad 1: /GND -> GND
- C100 pad 2: /XTALO -> XTALO
- C101 pad 1: /GND -> GND
- C102 pad 1: /GND -> GND
- C103 pad 1: /GND -> GND
- C103 pad 2: /SD_VCC -> SD_VCC
- C104 pad 1: /GND -> GND
- C104 pad 2: /SD_VCC -> SD_VCC
- C105 pad 1: /GND -> GND
- C106 pad 1: /GND -> GND
- C107 pad 1: /GND -> GND
- C108 pad 1: /GND -> GND
- C109 pad 1: /GND -> GND
- C11 pad 1: /GND -> GND
- C11 pad 2: /V+ -> V+
- C115 pad 1: /GND -> GND
- C116 pad 2: /GND -> GND
- C117 pad 1: /GND -> GND
- C117 pad 2: /VCC -> VCC
- C118 pad 1: /GND -> GND
- C118 pad 2: /VCC -> VCC
- C119 pad 1: /GND -> GND
- C119 pad 2: /VCC -> VCC
- C12 pad 1: /GND -> GND
- C120 pad 1: /GND -> GND
- C121 pad 1: /GND -> GND
- C122 pad 2: /GND -> GND
- C123 pad -: /GND -> GND
- C124 pad 2: /GND -> GND
- C125 pad 2: /GND -> GND
- C126 pad -: /GND -> GND
- C127 pad 1: /GND -> GND
- C128 pad 2: /GND -> GND
- C129 pad 1: /GND -> GND
- C13 pad 1: /GND -> GND
- C130 pad 2: /GND -> GND
- C131 pad 1: /GND -> GND
- C132 pad 1: /GND -> GND
- C133 pad 1: /GND -> GND
- C134 pad 1: /GND -> GND
- C135 pad -: /GND -> GND
- C136 pad 2: /GND -> GND
- C137 pad 2: /GND -> GND
- C138 pad 1: /GND -> GND
- C139 pad 1: /GND -> GND
- C14 pad 1: /GND -> GND
- C144 pad 2: /GND -> GND
- C145 pad 1: /GND -> GND
- C146 pad 1: /GND -> GND
- C149 pad 1: /GND -> GND
- C15 pad 1: /GND -> GND
- C151 pad 2: /GND -> GND
- C152 pad 2: /GND -> GND
- C153 pad 2: /GND -> GND
- C154 pad 2: /GND -> GND
- C155 pad 2: /GND -> GND
- C156 pad 2: /GND -> GND
- C157 pad 1: /GND -> GND
- C158 pad 1: /GND -> GND
- C159 pad 1: /VCC/2 -> VCC/2
- C159 pad 2: /GND -> GND
- C16 pad 1: /GND -> GND
- C160 pad 1: /VCC/2 -> VCC/2
- C160 pad 2: /GND -> GND
- C162 pad 2: /GND -> GND
- C163 pad 1: /GND -> GND
- C164 pad 1: /VCCINT -> VCCINT
- C164 pad 2: /GND -> GND
- C165 pad 1: /VCCINT -> VCCINT
- C165 pad 2: /GND -> GND
- C166 pad 2: /GND -> GND
- C167 pad 1: /GND -> GND
- C168 pad 1: /GND -> GND
- C169 pad 1: /GND -> GND
- C17 pad 1: /V+ -> V+
- C170 pad 1: /GND -> GND
- C171 pad 1: /GND -> GND
- C172 pad 2: /GND -> GND
- C173 pad 1: /GND -> GND
- C174 pad 1: /GND -> GND
- C175 pad 1: /GND -> GND
- C176 pad 1: /GND -> GND
- C177 pad 1: /GND -> GND
- C178 pad 2: /GND -> GND
- C179 pad 2: /GND -> GND
- C18 pad 1: /GND -> GND
- C18 pad 2: /VCCINT -> VCCINT
- C180 pad 2: /GND -> GND
- C181 pad 1: /GND -> GND
- C182 pad 1: /GND -> GND
- C183 pad 1: /GND -> GND
- C184 pad 2: /GND -> GND
- C185 pad 1: /GND -> GND
- C186 pad 1: /GND -> GND
- C187 pad 2: /GND -> GND
- C188 pad 1: /GND -> GND
- C189 pad 2: /GND -> GND
- C19 pad 1: /GND -> GND
- C19 pad 2: /VCCINT -> VCCINT
- C190 pad 1: /GND -> GND
- C191 pad 2: /GND -> GND
- C192 pad 1: /GND -> GND
- C193 pad 1: /GND -> GND
- C194 pad 2: /GND -> GND
- C195 pad 1: /V+ -> V+
- C196 pad 1: /GND -> GND
- C197 pad 1: /GND -> GND
- C198 pad 1: /V+ -> V+
- C198 pad 2: /GND -> GND
- C199 pad 1: /V+ -> V+
- C199 pad 2: /GND -> GND
- C2 pad 1: /GND -> GND
- C2 pad 2: /V+ -> V+
- C20 pad 1: /GND -> GND
- C20 pad 2: /VCCINT -> VCCINT
- C202 pad -: /GND -> GND
- C203 pad 2: /GND -> GND
- C204 pad 2: /GND -> GND
- C205 pad 2: /GND -> GND
- C206 pad 2: /GND -> GND
- C207 pad 2: /GND -> GND
- C208 pad 1: /VCC -> VCC
- C209 pad 1: /GND -> GND
- C21 pad 1: /GND -> GND
- C21 pad 2: /VCCINT -> VCCINT
- C210 pad 1: /GND -> GND
- C211 pad 1: /VCC -> VCC
- C211 pad 2: /GND -> GND
- C212 pad 1: /VCC -> VCC
- C212 pad 2: /GND -> GND
- C213 pad 1: /GND -> GND
- C214 pad 1: /GND -> GND
- C215 pad 1: /GND -> GND
- C216 pad 2: /GND -> GND
- C218 pad 2: /GND -> GND
- C219 pad 1: /VCC -> VCC
- C219 pad 2: /GND -> GND
- C22 pad 1: /GND -> GND
- C22 pad 2: /VCCINT -> VCCINT
- C220 pad 2: /GND -> GND
- C221 pad 2: /GND -> GND
- C224 pad 1: /GND -> GND
- C224 pad 2: /V+ -> V+
- C225 pad 1: /GND -> GND
- C225 pad 2: /V+ -> V+
- C226 pad 1: /GND -> GND
- C226 pad 2: /V+ -> V+
- C227 pad 1: /GND -> GND
- C227 pad 2: /V+ -> V+
- C228 pad 1: /GND -> GND
- C228 pad 2: /V+ -> V+
- C229 pad 1: /GND -> GND
- C229 pad 2: /V+ -> V+
- C23 pad 1: /GND -> GND
- C23 pad 2: /VCCINT -> VCCINT
- C230 pad 1: /GND -> GND
- C230 pad 2: /V+ -> V+
- C231 pad 1: /GND -> GND
- C231 pad 2: /V+ -> V+
- C232 pad 1: /GND -> GND
- C232 pad 2: /V+ -> V+
- C24 pad 1: /GND -> GND
- C24 pad 2: /VCCINT -> VCCINT
- C25 pad 1: /GND -> GND
- C25 pad 2: /VCCINT -> VCCINT
- C26 pad 1: /GND -> GND
- C26 pad 2: /VCCINT -> VCCINT
- C27 pad 1: /GND -> GND
- C27 pad 2: /VCCINT -> VCCINT
- C28 pad 1: /GND -> GND
- C28 pad 2: /V+ -> V+
- C29 pad 1: /GND -> GND
- C29 pad 2: /V+ -> V+
- C3 pad 1: /GND -> GND
- C3 pad 2: /V+ -> V+
- C30 pad 1: /GND -> GND
- C30 pad 2: /V+ -> V+
- C31 pad 1: /GND -> GND
- C31 pad 2: /V+ -> V+
- C32 pad 1: /GND -> GND
- C32 pad 2: /V+ -> V+
- C33 pad 1: /GND -> GND
- C33 pad 2: /V+ -> V+
- C34 pad 1: /GND -> GND
- C34 pad 2: /V+ -> V+
- C35 pad 1: /GND -> GND
- C36 pad 1: /GND -> GND
- C36 pad 2: /V+ -> V+
- C37 pad 1: /GND -> GND
- C37 pad 2: /V+ -> V+
- C38 pad 1: /GND -> GND
- C38 pad 2: /V+ -> V+
- C39 pad 1: /GND -> GND
- C39 pad 2: /V+ -> V+
- C4 pad 1: /GND -> GND
- C4 pad 2: /V+ -> V+
- C40 pad 1: /GND -> GND
- C40 pad 2: /V+ -> V+
- C41 pad 1: /GND -> GND
- C41 pad 2: /V+ -> V+
- C42 pad 1: /GND -> GND
- C42 pad 2: /V+ -> V+
- C43 pad 1: /GND -> GND
- C43 pad 2: /V+ -> V+
- C44 pad 1: /GND -> GND
- C44 pad 2: /V+ -> V+
- C45 pad 1: /GND -> GND
- C45 pad 2: /V+ -> V+
- C46 pad 1: /GND -> GND
- C46 pad 2: /V+ -> V+
- C47 pad 1: /GND -> GND
- C47 pad 2: /V+ -> V+
- C48 pad 1: /GND -> GND
- C48 pad 2: /V+ -> V+
- C49 pad 1: /GND -> GND
- C49 pad 2: /V+ -> V+
- C5 pad 1: /GND -> GND
- C5 pad 2: /V+ -> V+
- C50 pad 1: /GND -> GND
- C50 pad 2: /V+ -> V+
- C51 pad 1: /GND -> GND
- C51 pad 2: /V+ -> V+
- C52 pad 1: /GND -> GND
- C52 pad 2: /V+ -> V+
- C53 pad 1: /GND -> GND
- C53 pad 2: /V+ -> V+
- C54 pad 1: /GND -> GND
- C54 pad 2: /V+ -> V+
- C55 pad 1: /GND -> GND
- C55 pad 2: /V+ -> V+
- C56 pad 1: /GND -> GND
- C57 pad 1: /GND -> GND
- C57 pad 2: /VCC/2 -> VCC/2
- C58 pad 1: /GND -> GND
- C58 pad 2: /VCC/2 -> VCC/2
- C59 pad 1: /GND -> GND
- C59 pad 2: /VCC/2 -> VCC/2
- C6 pad 1: /GND -> GND
- C6 pad 2: /V+ -> V+
- C60 pad 1: /GND -> GND
- C60 pad 2: /VCC/2 -> VCC/2
- C61 pad 1: /GND -> GND
- C61 pad 2: /VCC/2 -> VCC/2
- C62 pad 1: /GND -> GND
- C62 pad 2: /VCC/2 -> VCC/2
- C63 pad 1: /GND -> GND
- C64 pad 1: /GND -> GND
- C65 pad 1: /GND -> GND
- C66 pad 1: /GND -> GND
- C67 pad 1: /GND -> GND
- C68 pad 1: /GND -> GND
- C68 pad 2: /VCC -> VCC
- C69 pad 1: /GND -> GND
- C69 pad 2: /VCC -> VCC
- C7 pad 1: /GND -> GND
- C7 pad 2: /V+ -> V+
- C70 pad 1: /GND -> GND
- C70 pad 2: /VCC -> VCC
- C71 pad 1: /GND -> GND
- C72 pad 1: /GND -> GND
- C72 pad 2: /XTALI1 -> XTALI1
- C73 pad 1: /GND -> GND
- C73 pad 2: /XTALO1 -> XTALO1
- C74 pad 2: /GND -> GND
- C75 pad 2: /GND -> GND
- C76 pad 2: /GND -> GND
- C77 pad 1: /GND -> GND
- C77 pad 2: /VCC -> VCC
- C78 pad 1: /GND -> GND
- C78 pad 2: /VCC -> VCC
- C79 pad 1: /GND -> GND
- C79 pad 2: /VCC -> VCC
- C8 pad 1: /GND -> GND
- C8 pad 2: /V+ -> V+
- C80 pad 1: /GND -> GND
- C80 pad 2: /VCC -> VCC
- C81 pad 1: /GND -> GND
- C81 pad 2: /VCC -> VCC
- C82 pad 1: /GND -> GND
- C82 pad 2: /VCC -> VCC
- C83 pad 1: /GND -> GND
- C83 pad 2: /VCC -> VCC
- C84 pad 1: /GND -> GND
- C84 pad 2: /VCC -> VCC
- C85 pad 1: /GND -> GND
- C85 pad 2: /VCC -> VCC
- C86 pad 1: /GND -> GND
- C87 pad 1: /GND -> GND
- C88 pad 1: /GND -> GND
- C89 pad 1: /GND -> GND
- C89 pad 2: /VCC -> VCC
- C9 pad 1: /GND -> GND
- C9 pad 2: /V+ -> V+
- C90 pad 1: /GND -> GND
- C90 pad 2: /VCC -> VCC
- C91 pad 1: /GND -> GND
- C92 pad 1: /GND -> GND
- C93 pad 1: /GND -> GND
- C94 pad 1: /GND -> GND
- C95 pad 1: /GND -> GND
- C96 pad 1: /GND -> GND
- C97 pad 1: /GND -> GND
- C98 pad 1: /GND -> GND
- C99 pad 1: /GND -> GND
- C99 pad 2: /XTALI -> XTALI
- D1 pad A: /VCC -> VCC
- D5 pad A: /GND -> GND
- ENTER233 pad 2_1: /GND -> GND
- ESC233 pad 2_1: /GND -> GND
- FET2 pad 2: /GND -> GND
- FET3 pad 2: /GND -> GND
- GND233 pad 1: /GND -> GND
- GND_PIN233 pad P$1: /GND -> GND
- GPIO-1 pad 2: /GND -> GND
- GPIO-1 pad 3: /VCC -> VCC
- GPIO-1 pad 4: /GND -> GND
- GPIO-2 pad 2: /GND -> GND
- GPIO-2 pad 3: /VCC -> VCC
- GPIO-2 pad 4: /GND -> GND
- GPIO-3 pad 2: /GND -> GND
- GPIO-3 pad 3: /VCC -> VCC
- GPIO-3 pad 4: /GND -> GND
- HDMI233 pad 11: /GND -> GND
- HDMI233 pad 14: Net-(HDMI233-Pad14) -> (no net)
- HDMI233 pad 17: /GND -> GND
- HDMI233 pad 2: /GND -> GND
- HDMI233 pad 5: /GND -> GND
- HDMI233 pad 8: /GND -> GND
- HDMI233 pad SH1: /GND -> GND
- HDMI233 pad SH2: /GND -> GND
- HDMI233 pad SH3: /GND -> GND
- HDMI233 pad SH4: /GND -> GND
- HEADPHONES233 pad 1: Net-(HEADPHONES233-Pad1) -> (no net)
- HEADPHONES233 pad 4: Net-(HEADPHONES233-Pad4) -> (no net)
- HOME233 pad 2_1: /GND -> GND
- L1 pad 2: /VCC -> VCC
- L11 pad 1: /GND -> GND
- L13 pad 2: /VCC/2 -> VCC/2
- L14 pad 2: /VCCINT -> VCCINT
- L18 pad 2: /V+ -> V+
- L2 pad 2: /VCC -> VCC
- L21 pad 2: /VCC -> VCC
- L4 pad 1: /VCC -> VCC
- L4 pad 2: /SD_VCC -> SD_VCC
- L5 pad 1: /VCC -> VCC
- L7 pad 1: /GND -> GND
- LAN233 pad 6: Net-(LAN233-Pad6) -> (no net)
- LAN233 pad AG: /VCC -> VCC
- LAN233 pad GND1: /GND -> GND
- LAN233 pad GND2: /GND -> GND
- LCD_CON233 pad 2: /GND -> GND
- LCD_CON233 pad 3: /VCC -> VCC
- LCD_CON233 pad 4: /GND -> GND
- LED1 pad C: /GND -> GND
- LIPO_BAT233 pad 2: /GND -> GND
- MENU233 pad 2_1: /GND -> GND
- MIC_IN233 pad 1: Net-(MIC_IN233-Pad1) -> (no net)
- MIC_IN233 pad 4: Net-(MIC_IN233-Pad4) -> (no net)
- MIC_IN233 pad 5: /GND -> GND
- PWR233 pad -: /GND -> GND
- PWR233 pad --: /GND -> GND
- PWR_BUT233 pad 2_1: /GND -> GND
- PWR_LED233 pad C: /GND -> GND
- Q2 pad GND: /GND -> GND
- R1 pad 2: /V+ -> V+
- R10 pad 2: /VCC -> VCC
- R105 pad 2: /VCC -> VCC
- R11 pad 2: /VCC -> VCC
- R120 pad 2: /GND -> GND
- R121 pad 1: /VCC -> VCC
- R125 pad 1: /VCC -> VCC
- R13 pad 1: /VCC -> VCC
- R130 pad 1: /VCC -> VCC
- R138 pad 1: /GND -> GND
- R14 pad 2: /VCC -> VCC
- R16 pad 1: /GND -> GND
- R18 pad 1: /VCC -> VCC
- R19 pad 1: /VCC -> VCC
- R2 pad 1: /GND -> GND
- R20 pad 1: /GND -> GND
- R21 pad 1: /VCC -> VCC
- R24 pad 1: /GND -> GND
- R26 pad 2: /GND -> GND
- R28 pad 2: /VCC -> VCC
- R29 pad 1: /SD0-D3 -> SD0-D3
- R29 pad 2: /VCC -> VCC
- R3 pad 2: /VCCINT -> VCCINT
- R30 pad 1: /SD0-CMD -> SD0-CMD
- R30 pad 2: /VCC -> VCC
- R31 pad 2: /VCC -> VCC
- R33 pad 1: /N$58 -> N$58
- R33 pad 2: /GND -> GND
- R35 pad 2: /GND -> GND
- R4 pad 2: /V+ -> V+
- R40 pad 2: /GND -> GND
- R44 pad 1: /GND -> GND
- R45 pad 1: /GND -> GND
- R46 pad 1: /GND -> GND
- R47 pad 1: /GND -> GND
- R48 pad 1: /GND -> GND
- R51 pad 2: /VCC -> VCC
- R52 pad 1: /VCC -> VCC
- R53 pad 2: /VCCINT -> VCCINT
- R54 pad 1: /GND -> GND
- R55 pad 1: /GND -> GND
- R56 pad 2: /GND -> GND
- R58 pad 1: /GND -> GND
- R6 pad 2: /V+ -> V+
- R60 pad 1: /VCC -> VCC
- R64 pad 1: /GND -> GND
- R67 pad 1: /GND -> GND
- R68 pad 2: /VCCINT -> VCCINT
- R7 pad 1: /GND -> GND
- R72 pad 1: /VCC -> VCC
- R73 pad 1: /GND -> GND
- R74 pad 1: /VCC -> VCC
- R75 pad 2: /VCC -> VCC
- R76 pad 2: /VCC -> VCC
- R77 pad 1: /V+ -> V+
- R78 pad 2: /GND -> GND
- R8 pad 1: /GND -> GND
- R82 pad 2: /VCC -> VCC
- R83 pad 2: /VCC -> VCC
- R84 pad 2: /VCC -> VCC
- R85 pad 2: /GND -> GND
- R86 pad 2: /GND -> GND
- R87 pad 1: /GND -> GND
- R89 pad 1: /VCC -> VCC
- R9 pad 1: /GND -> GND
- R90 pad 2: /GND -> GND
- R92 pad 2: /GND -> GND
- R93 pad 2: /VCC -> VCC
- R94 pad 2: /VCC -> VCC
- R95 pad 2: /VCC -> VCC
- RECOVERY233 pad 1_1: /GND -> GND
- RM10 pad 1.2: /VCC -> VCC
- RM10 pad 2.2: /VCC -> VCC
- RM10 pad 3.2: /GND -> GND
- RM14 pad 1.1: /VCC -> VCC
- RM14 pad 1.2: /SD0-D2 -> SD0-D2
- RM14 pad 2.1: /VCC -> VCC
- RM14 pad 2.2: /SD0-D0 -> SD0-D0
- RM14 pad 3.1: /VCC -> VCC
- RM14 pad 3.2: /SD0-D1 -> SD0-D1
- RM14 pad 4.1: /VCC -> VCC
- RM14 pad 4.2: /SD0-DET# -> SD0-DET#
- RM15 pad 1.2: /VCC -> VCC
- RM15 pad 2.2: /VCC -> VCC
- RM15 pad 3.2: /VCC -> VCC
- RM15 pad 4.2: /VCC -> VCC
- RM24 pad 2.1: /GND -> GND
- RM24 pad 3.1: /GND -> GND
- RM24 pad 4.1: /GND -> GND
- RM25 pad 1.2: /VCC -> VCC
- RM25 pad 2.2: /VCC -> VCC
- RM25 pad 3.2: /VCC -> VCC
- RM9 pad 1.1: /VCC -> VCC
- RM9 pad 2.1: /GND -> GND
- RM9 pad 3.1: /GND -> GND
- RM9 pad 4.1: /GND -> GND
- SATA233 pad 1: /GND -> GND
- SATA233 pad 4: /GND -> GND
- SATA233 pad 7: /GND -> GND
- SD/MMC2 pad 3: /GND -> GND
- SD/MMC2 pad 6: /GND -> GND
- SD/MMC2 pad SH1: /GND -> GND
- SD/MMC2 pad SH2: /GND -> GND
- SD/MMC2 pad WP: /GND -> GND
- SEARCH233 pad 2_1: /GND -> GND
- T1 pad 2: /GND -> GND
- U1 pad AA18: /GND -> GND
- U1 pad AB19: /VCC -> VCC
- U1 pad B6: /SD0-DET# -> SD0-DET#
- U1 pad G3: /GND -> GND
- U1 pad G4: /GND -> GND
- U1 pad G5: /V+ -> V+
- U1 pad H10: /VCC -> VCC
- U1 pad H11: /VCC/2 -> VCC/2
- U1 pad H12: /VCC/2 -> VCC/2
- U1 pad H13: /VCC/2 -> VCC/2
- U1 pad H14: /VCC/2 -> VCC/2
- U1 pad H15: /VCC -> VCC
- U1 pad H16: /GND -> GND
- U1 pad H19: /VCC -> VCC
- U1 pad H5: /V+ -> V+
- U1 pad H8: /VCC -> VCC
- U1 pad H9: /VCC -> VCC
- U1 pad J10: /VCC -> VCC
- U1 pad J11: /GND -> GND
- U1 pad J12: /VCC/2 -> VCC/2
- U1 pad J13: /VCC/2 -> VCC/2
- U1 pad J14: /VCC -> VCC
- U1 pad J15: /VCCINT -> VCCINT
- U1 pad J16: /VCCINT -> VCCINT
- U1 pad J19: /VCC -> VCC
- U1 pad J5: /GND -> GND
- U1 pad J8: /VCC -> VCC
- U1 pad J9: /VCC -> VCC
- U1 pad K10: /VCCINT -> VCCINT
- U1 pad K11: /GND -> GND
- U1 pad K12: /GND -> GND
- U1 pad K13: /GND -> GND
- U1 pad K14: /GND -> GND
- U1 pad K15: /VCCINT -> VCCINT
- U1 pad K19: /SD0-D2 -> SD0-D2
- U1 pad K20: /SD0-D3 -> SD0-D3
- U1 pad K5: /GND -> GND
- U1 pad K9: /VCCINT -> VCCINT
- U1 pad L10: /GND -> GND
- U1 pad L11: /GND -> GND
- U1 pad L12: /GND -> GND
- U1 pad L13: /GND -> GND
- U1 pad L14: /GND -> GND
- U1 pad L19: /SD0-CMD -> SD0-CMD
- U1 pad L20: /SD0-CLK -> SD0-CLK
- U1 pad L5: /V+ -> V+
- U1 pad L8: /VCCINT -> VCCINT
- U1 pad L9: /VCCINT -> VCCINT
- U1 pad M10: /GND -> GND
- U1 pad M11: /GND -> GND
- U1 pad M12: /GND -> GND
- U1 pad M13: /GND -> GND
- U1 pad M14: /GND -> GND
- U1 pad M19: /SD0-D0 -> SD0-D0
- U1 pad M20: /SD0-D1 -> SD0-D1
- U1 pad M5: /V+ -> V+
- U1 pad M9: /GND -> GND
- U1 pad N10: /GND -> GND
- U1 pad N11: /GND -> GND
- U1 pad N12: /GND -> GND
- U1 pad N13: /GND -> GND
- U1 pad N14: /GND -> GND
- U1 pad N19: /VCC -> VCC
- U1 pad N22: /XTALO -> XTALO
- U1 pad N23: /XTALI -> XTALI
- U1 pad N5: /GND -> GND
- U1 pad P10: /GND -> GND
- U1 pad P11: /GND -> GND
- U1 pad P12: /GND -> GND
- U1 pad P13: /GND -> GND
- U1 pad P14: /GND -> GND
- U1 pad P15: /GND -> GND
- U1 pad P19: Net-(U1-PadP19) -> (no net)
- U1 pad P5: /GND -> GND
- U1 pad R10: /VCCINT -> VCCINT
- U1 pad R11: /GND -> GND
- U1 pad R12: /GND -> GND
- U1 pad R13: /GND -> GND
- U1 pad R16: Net-(U1-PadR16) -> (no net)
- U1 pad R19: Net-(U1-PadR19) -> (no net)
- U1 pad R5: /V+ -> V+
- U1 pad R9: /VCCINT -> VCCINT
- U1 pad T11: /GND -> GND
- U1 pad T12: /GND -> GND
- U1 pad T15: Net-(U1-PadT15) -> (no net)
- U1 pad T5: /V+ -> V+
- U1 pad T8: /VCCINT -> VCCINT
- U1 pad U19: /GND -> GND
- U1 pad U5: /GND -> GND
- U1 pad V19: /GND -> GND
- U1 pad V5: /GND -> GND
- U1 pad W10: /GND -> GND
- U1 pad W11: /GND -> GND
- U1 pad W12: /VCC -> VCC
- U1 pad W13: /VCC -> VCC
- U1 pad W14: /VCC -> VCC
- U1 pad W18: /GND -> GND
- U1 pad W5: /V+ -> V+
- U1 pad W6: /V+ -> V+
- U1 pad W7: /V+ -> V+
- U1 pad W9: /GND -> GND
- U1 pad Y18: /GND -> GND
- U1 pad Y6: /V+ -> V+
- U1 pad Y7: /GND -> GND
- U1 pad Y8: /GND -> GND
- U10 pad 2: /GND -> GND
- U11 pad 2: /GND -> GND
- U12 pad 10: /VCC/2 -> VCC/2
- U12 pad 16: /GND -> GND
- U12 pad 17: /VCCINT -> VCCINT
- U12 pad 22: /GND -> GND
- U12 pad 29: Net-(U12-Pad29) -> (no net)
- U12 pad 30: Net-(U12-Pad30) -> (no net)
- U12 pad 46: /GND -> GND
- U12 pad 9: /GND -> GND
- U12 pad N1: Net-(U12-PadN1) -> GND
- U12 pad N10: Net-(U12-PadN1) -> GND
- U12 pad N11: Net-(U12-PadN1) -> GND
- U12 pad N12: Net-(U12-PadN1) -> GND
- U12 pad N13: Net-(U12-PadN1) -> GND
- U12 pad N14: Net-(U12-PadN1) -> GND
- U12 pad N15: Net-(U12-PadN1) -> GND
- U12 pad N16: Net-(U12-PadN1) -> GND
- U12 pad N17: Net-(U12-PadN1) -> GND
- U12 pad N2: Net-(U12-PadN1) -> GND
- U12 pad N3: Net-(U12-PadN1) -> GND
- U12 pad N4: Net-(U12-PadN1) -> GND
- U12 pad N5: Net-(U12-PadN1) -> GND
- U12 pad N6: Net-(U12-PadN1) -> GND
- U12 pad N7: Net-(U12-PadN1) -> GND
- U12 pad N8: Net-(U12-PadN1) -> GND
- U12 pad N9: Net-(U12-PadN1) -> GND
- U12 pad VSS: /GND -> GND
- U13 pad 2: /GND -> GND
- U14 pad 4: /GND -> GND
- U15 pad 2: /GND -> GND
- U16 pad 2: /GND -> GND
- U16 pad 6: Net-(U16-Pad6) -> (no net)
- U17 pad 3: /GND -> GND
- U17 pad 8: /GND -> GND
- U2 pad A1: /V+ -> V+
- U2 pad A8: /V+ -> V+
- U2 pad A9: /GND -> GND
- U2 pad B1: /GND -> GND
- U2 pad B2: /V+ -> V+
- U2 pad B3: /GND -> GND
- U2 pad B9: /GND -> GND
- U2 pad C1: /V+ -> V+
- U2 pad C9: /V+ -> V+
- U2 pad D1: /GND -> GND
- U2 pad D2: /V+ -> V+
- U2 pad D8: /GND -> GND
- U2 pad D9: /V+ -> V+
- U2 pad E1: /GND -> GND
- U2 pad E2: /GND -> GND
- U2 pad E8: /GND -> GND
- U2 pad E9: /V+ -> V+
- U2 pad F1: /V+ -> V+
- U2 pad F9: /GND -> GND
- U2 pad G1: /GND -> GND
- U2 pad G7: /V+ -> V+
- U2 pad G8: /GND -> GND
- U2 pad G9: /GND -> GND
- U2 pad H2: /V+ -> V+
- U2 pad H9: /V+ -> V+
- U2 pad J1: Net-(U2-PadJ1) -> (no net)
- U2 pad J2: /GND -> GND
- U2 pad J8: /GND -> GND
- U2 pad J9: Net-(U2-PadJ9) -> (no net)
- U2 pad K2: /V+ -> V+
- U2 pad K8: /V+ -> V+
- U2 pad L1: Net-(U2-PadL1) -> (no net)
- U2 pad L9: Net-(U2-PadL9) -> (no net)
- U2 pad M1: /GND -> GND
- U2 pad M9: /GND -> GND
- U2 pad N1: /V+ -> V+
- U2 pad N9: /V+ -> V+
- U2 pad P1: /GND -> GND
- U2 pad P9: /GND -> GND
- U2 pad R1: /V+ -> V+
- U2 pad R9: /V+ -> V+
- U2 pad T1: /GND -> GND
- U2 pad T9: /GND -> GND
- U22 pad 3: /GND -> GND
- U22 pad 8: /GND -> GND
- U23 pad 3: /GND -> GND
- U23 pad 8: /GND -> GND
- U3 pad A1: /V+ -> V+
- U3 pad A8: /V+ -> V+
- U3 pad A9: /GND -> GND
- U3 pad B1: /GND -> GND
- U3 pad B2: /V+ -> V+
- U3 pad B3: /GND -> GND
- U3 pad B9: /GND -> GND
- U3 pad C1: /V+ -> V+
- U3 pad C9: /V+ -> V+
- U3 pad D1: /GND -> GND
- U3 pad D2: /V+ -> V+
- U3 pad D8: /GND -> GND
- U3 pad D9: /V+ -> V+
- U3 pad E1: /GND -> GND
- U3 pad E2: /GND -> GND
- U3 pad E8: /GND -> GND
- U3 pad E9: /V+ -> V+
- U3 pad F1: /V+ -> V+
- U3 pad F9: /GND -> GND
- U3 pad G1: /GND -> GND
- U3 pad G7: /V+ -> V+
- U3 pad G8: /GND -> GND
- U3 pad G9: /GND -> GND
- U3 pad H2: /V+ -> V+
- U3 pad H9: /V+ -> V+
- U3 pad J1: Net-(U3-PadJ1) -> (no net)
- U3 pad J2: /GND -> GND
- U3 pad J8: /GND -> GND
- U3 pad J9: Net-(U3-PadJ9) -> (no net)
- U3 pad K2: /V+ -> V+
- U3 pad K8: /V+ -> V+
- U3 pad L1: Net-(U3-PadL1) -> (no net)
- U3 pad L9: Net-(U3-PadL9) -> (no net)
- U3 pad M1: /GND -> GND
- U3 pad M9: /GND -> GND
- U3 pad N1: /V+ -> V+
- U3 pad N9: /V+ -> V+
- U3 pad P1: /GND -> GND
- U3 pad P9: /GND -> GND
- U3 pad R1: /V+ -> V+
- U3 pad R9: /V+ -> V+
- U3 pad T1: /GND -> GND
- U3 pad T9: /GND -> GND
- U6 pad 1: /GND -> GND
- U6 pad 2: /GND -> GND
- U6 pad 3: /GND -> GND
- U6 pad 4: /GND -> GND
- U6 pad 7: /GND -> GND
- U6 pad 8: /VCC -> VCC
- U7 pad 11: /GND -> GND
- U7 pad 17: /GND -> GND
- U7 pad 27: Net-(U7-Pad27) -> (no net)
- U7 pad 29: /GND -> GND
- U7 pad 35: /GND -> GND
- U7 pad 37: /VCC -> VCC
- U7 pad 38: /VCC -> VCC
- U7 pad 39: /VCC -> VCC
- U7 pad 40: /GND -> GND
- U7 pad 41: /VCC -> VCC
- U7 pad 43: /GND -> GND
- U7 pad 44: /VCC -> VCC
- U7 pad 45: /GND -> GND
- U7 pad 46: /XTALI1 -> XTALI1
- U7 pad 47: /XTALO1 -> XTALO1
- U8 pad 1: /VCC -> VCC
- U8 pad 11: Net-(U8-Pad11) -> (no net)
- U8 pad 12: /VCC -> VCC
- U8 pad 13: /GND -> GND
- U8 pad 14: Net-(U8-Pad14) -> (no net)
- U8 pad 15: Net-(U8-Pad15) -> (no net)
- U8 pad 2: /GND -> GND
- U8 pad 20: Net-(U8-Pad20) -> (no net)
- U8 pad 21: Net-(U8-Pad21) -> (no net)
- U8 pad 22: Net-(U8-Pad22) -> (no net)
- U8 pad 23: /GND -> GND
- U8 pad 24: /VCC -> VCC
- U8 pad 25: /GND -> GND
- U8 pad 3: Net-(U8-Pad3) -> (no net)
- U8 pad 34: /VCC -> VCC
- U8 pad 36: /GND -> GND
- U8 pad 37: /VCC -> VCC
- U8 pad 39: /VCC -> VCC
- U8 pad 48: /GND -> GND
- U9 pad 2: /GND -> GND
- UART0 pad 1: /VCC -> VCC
- UART0 pad 4: /GND -> GND
- UEXT1 pad 1: /VCC -> VCC
- UEXT1 pad 2: /GND -> GND
- UEXT2 pad 1: /VCC -> VCC
- UEXT2 pad 2: /GND -> GND
- USB_HOST233 pad 1.4: /GND -> GND
- USB_HOST233 pad 2.4: /GND -> GND
- USB_OTG233 pad GND: /GND -> GND
- VGA233 pad 6: /GND -> GND
- VOL+233 pad 2_1: /GND -> GND
- VOL-233 pad 2_1: /GND -> GND
- VPS+233 pad 1: /VCC -> VCC
- VPS-233 pad 1: /GND -> GND
- VP_0 pad VP: /GND -> GND
- VP_1 pad VP: /GND -> GND
- VP_10 pad VP: /GND -> GND
- VP_11 pad VP: /GND -> GND
- VP_12 pad VP: /GND -> GND
- VP_13 pad VP: /GND -> GND
- VP_14 pad VP: /GND -> GND
- VP_15 pad VP: /GND -> GND
- VP_16 pad VP: /GND -> GND
- VP_17 pad VP: /GND -> GND
- VP_18 pad VP: /GND -> GND
- VP_19 pad VP: /GND -> GND
- VP_2 pad VP: /GND -> GND
- VP_20 pad VP: /GND -> GND
- VP_21 pad VP: /GND -> GND
- VP_22 pad VP: /GND -> GND
- VP_23 pad VP: /GND -> GND
- VP_24 pad VP: /GND -> GND
- VP_25 pad VP: /GND -> GND
- VP_26 pad VP: /GND -> GND
- VP_27 pad VP: /GND -> GND
- VP_28 pad VP: /GND -> GND
- VP_29 pad VP: /GND -> GND
- VP_3 pad VP: /GND -> GND
- VP_30 pad VP: /GND -> GND
- VP_31 pad VP: /GND -> GND
- VP_32 pad VP: /GND -> GND
- VP_33 pad VP: /GND -> GND
- VP_34 pad VP: /GND -> GND
- VP_35 pad VP: /GND -> GND
- VP_36 pad VP: /GND -> GND
- VP_37 pad VP: /GND -> GND
- VP_38 pad VP: /GND -> GND
- VP_39 pad VP: /GND -> GND
- VP_4 pad VP: /GND -> GND
- VP_40 pad VP: /GND -> GND
- VP_41 pad VP: /GND -> GND
- VP_42 pad VP: /GND -> GND
- VP_43 pad VP: /GND -> GND
- VP_44 pad VP: /GND -> GND
- VP_45 pad VP: /GND -> GND
- VP_46 pad VP: /GND -> GND
- VP_47 pad VP: /GND -> GND
- VP_48 pad VP: /GND -> GND
- VP_49 pad VP: /GND -> GND
- VP_5 pad VP: /GND -> GND
- VP_50 pad VP: /GND -> GND
- VP_51 pad VP: /GND -> GND
- VP_52 pad VP: /GND -> GND
- VP_53 pad VP: /GND -> GND
- VP_54 pad VP: /GND -> GND
- VP_55 pad VP: /GND -> GND
- VP_6 pad VP: /GND -> GND
- VP_7 pad VP: /GND -> GND
- VP_8 pad VP: /GND -> GND
- VP_9 pad VP: /GND -> GND
- VR1 pad 1: /VCC -> VCC
- VR1 pad 2: /GND -> GND
- VR1 pad 3: /VCC -> VCC
Routing:
- net GND: track 1.40 -> 693.5 mm, vias 1 -> 255
- net /GND: track 666.6 -> 0.00 mm, vias 254 -> 0
- net VCCINT: track 0.00 -> 268.8 mm, vias 0 -> 18
- net /VCCINT: track 268.8 -> 0.00 mm, vias 18 -> 0
- net VCC: track 0.00 -> 198.5 mm, vias 0 -> 58
- net /VCC: track 198.5 -> 0.00 mm, vias 58 -> 0
- net SD0-D3: track 1.56 -> 126.8 mm, vias 0 -> 2
- net /SD0-D3: track 125.3 -> 0.00 mm, vias 2 -> 0
- net SD0-D2: track 7.62 -> 124.9 mm, vias 1 -> 3
- net /SD0-D2: track 117.3 -> 0.00 mm, vias 2 -> 0
- net SD0-CLK: track 1.40 -> 118.3 mm, vias 1 -> 2
- net /SD0-CLK: track 116.9 -> 0.00 mm, vias 1 -> 0
- net /SD0-CMD: track 116.4 -> 0.00 mm, vias 1 -> 0
- net SD0-CMD: track 8.79 -> 125.2 mm, vias 1 -> 2
- net SD0-D0: track 1.56 -> 116.4 mm, vias 0 -> 2
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