File: examples/OLINUXINO/A10-A20-OLINUXINO-MICRO-4GB_Rev_D/kicad_files/A10-A20-OLINUXINO-MICRO-4GB_Rev_D.sch (KiCad schematic (older format))
At the start: 551 parts, among them Q1 4SB25.000F20E15/5x3.2mm/20ppm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, Q2 32768Hz/6pF, Q3 4SB24.000F20E15/5x3.2mm/20ppm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, T1 BC846B, U1 A10/A20, U10 SY6280, U11 SY6280, U12 AXP209(QFN48), U13 SY8008C(AA)C, U14 MP1482DS, U15 SY8008C(AA)C, U16 SY7208(SOT23-6), U17 RCLAMP0524P, U2 H5TQ2G63BFR_MEM4G16D3EABG-125, U22 RCLAMP0524P, U23 RCLAMP0524P, U3 H5TQ2G63BFR_MEM4G16D3EABG-125, U6 AT24C16BN-SH, U7 RTL8201CP, U8 H27UBG8T2BTR, U9 SY6280

Commit message: replace / in deice name with _, to Fix few problems
Parts:
- removed Q1: 4SB25.000F20E15/5x3.2mm/20ppm/20pF, CRYSTAL_HCX-4S, symbol CRYSTAL_HC49/S_E4SB25.000F20E15
- removed Q3: 4SB24.000F20E15/5x3.2mm/20ppm/20pF, CRYSTAL_HCX-4S, symbol CRYSTAL_HC49/S_E4SB25.000F20E15
- removed SD/MMC1: MICRO_SD/MMC_CP_NEWTFC-WPAPR-08, OLIMEX_CONNECTORS_TFC-WPAPR-08, symbol OLIMEX_CONNECTORS_MICRO_SD/MMC_CP_NEWTFC-WPAPR-08
- added Q1: 4SB25.000F20E15/5x3.2mm/20ppm/20pF, A10-A20-OLINUXINO-MICRO-4GB_Rev_D:CRYSTAL_HCX-4S, symbol CRYSTAL_HC49_S_E4SB25.000F20E15
- added Q3: 4SB24.000F20E15/5x3.2mm/20ppm/20pF, A10-A20-OLINUXINO-MICRO-4GB_Rev_D:CRYSTAL_HCX-4S, symbol CRYSTAL_HC49_S_E4SB25.000F20E15
- added SD/MMC1: MICRO_SD/MMC_CP_NEWTFC-WPAPR-08, A10-A20-OLINUXINO-MICRO-4GB_Rev_D:OLIMEX_CONNECTORS_TFC-WPAPR-08, symbol OLIMEX_CONNECTORS_MICRO_SD_MMC_CP_NEWTFC-WPAPR-08
Connections:
- wire segments 2487 -> 3124
