File: examples/PIXHAWK/kicad_files/PX4FMUv2.4_SS_1.sch (KiCad schematic (older format))
At the start: 8 parts, among them U101 STM32F4X7VX, U102 FM25V01, X101 3.2x2.5 mm / 24 MHz / 15 ppm

Commit message: force golbale netnames on, to get around fill/net problem
Parts:
- C101, C102, C103: footprint PX4FMUv2.4:PIXHAWK2_0402-CAP -> PIXHAWK2_0402-CAP
- R101, R102: footprint PX4FMUv2.4:PIXHAWK2_0402-RES -> PIXHAWK2_0402-RES
- U101: footprint PX4FMUv2.4:PIXHAWK2_TQFP100 -> PIXHAWK2_TQFP100
- U102: footprint PX4FMUv2.4:PIXHAWK2_SO08 -> PIXHAWK2_SO08
- X101: footprint PX4FMUv2.4:PIXHAWK2_OSCILLATOR-3.2X2.5 -> PIXHAWK2_OSCILLATOR-3.2X2.5
Connections:
- wire segments 111 -> 119
