File: examples/PIXHAWK/kicad_files/PX4FMUv2.4_SS_10.sch (KiCad schematic (older format))
At the start: 12 parts, among them U1001 BQ24313, U1002 MIC5332

Commit message: force golbale netnames on, to get around fill/net problem
Parts:
- C1001: footprint PX4FMUv2.4:PIXHAWK2_0805-CAP -> PIXHAWK2_0805-CAP
- C1002, C1005, C1008: footprint PX4FMUv2.4:PIXHAWK2_0402-CAP -> PIXHAWK2_0402-CAP
- C1003, C1004: footprint PX4FMUv2.4:PIXHAWK2_0603-CAP -> PIXHAWK2_0603-CAP
- D1001: footprint PX4FMUv2.4:PIXHAWK2_SOT23-3 -> PIXHAWK2_SOT23-3
- F1001: footprint PX4FMUv2.4:PIXHAWK2_PTC-1206 -> PIXHAWK2_PTC-1206
- R1001, R1002: footprint PX4FMUv2.4:PIXHAWK2_0402-RES -> PIXHAWK2_0402-RES
- U1001: footprint PX4FMUv2.4:PIXHAWK2_QFN8-DSG -> PIXHAWK2_QFN8-DSG
- U1002: footprint PX4FMUv2.4:PIXHAWK2_MLF-8-EPAD -> PIXHAWK2_MLF-8-EPAD
Connections:
- wire segments 41 -> 50
