File: examples/PIXHAWK/kicad_files/PX4FMUv2.4_SS_11.sch (KiCad schematic (older format))
At the start: 32 parts, among them J601 DF13C-6P-1.25V, U1101 LTC4417, U1102 NTHD4102PT1G, U1103 NTHD4102PT1G, U1104 NTHD4102PT1G

Commit message: force golbale netnames on, to get around fill/net problem
Parts:
- C1101, C1102, C1103: footprint PX4FMUv2.4:PIXHAWK2_0805-CAP -> PIXHAWK2_0805-CAP
- C1104: footprint PX4FMUv2.4:PIXHAWK2_1206-CAP -> PIXHAWK2_1206-CAP
- C1105, C1106, C1107, C1108, C1109, C1110: footprint PX4FMUv2.4:PIXHAWK2_0402-CAP -> PIXHAWK2_0402-CAP
- J601: footprint PX4FMUv2.4:CON-HIROSE-DF13_DF13C-6P-1.25V -> CON-HIROSE-DF13_DF13C-6P-1.25V
- L1101, L1102: footprint PX4FMUv2.4:PIXHAWK2_KYOCERA-KNH16-DA -> PIXHAWK2_KYOCERA-KNH16-DA
- R1101, R1102, R1103, R1104, R1105, R1106, R1107, R1109, R1110, R1111, R1112, R1113, R1114, R1115: footprint PX4FMUv2.4:PIXHAWK2_0402-RES -> PIXHAWK2_0402-RES
- RN1101: footprint PX4FMUv2.4:RESISTOR-DIL_EXB28V -> RESISTOR-DIL_EXB28V
- U1101: footprint PX4FMUv2.4:PIXHAWK2_MO-220 -> PIXHAWK2_MO-220
- U1102, U1103, U1104: footprint PX4FMUv2.4:PIXHAWK2_1206-8 -> PIXHAWK2_1206-8; Field5 D -> (none); Field6 S -> (none); Field7 G -> (none)
Connections:
- wire segments 129 -> 180
