File: examples/PIXHAWK/kicad_files/PX4FMUv2.4_SS_12.sch (KiCad schematic (older format))
At the start: 95 parts, among them M3_MOUNT1101 MOUNT-HOLE3.1MM, M3_MOUNT1102 MOUNT-HOLE3.1MM, M3_MOUNT1103 MOUNT-HOLE3.1MM, M3_MOUNT1104 MOUNT-HOLE3.1MM

Commit message: force golbale netnames on, to get around fill/net problem
Parts:
- !VBUS_VALID1116, !VDD_BRICK_VALID1116, !VDD_SERVO_VALID1116, ADC_PR1116, CAN_H1116, CAN_L1116, FMU-BOOT1101, GND.1116, GND1116, IO-BOOT1101, S1RX1116, S1TX1116, S2RX1116, S2TX1116, S3RX1116, S3TX1116, S4RX1116, S4TX1116, S5_RX1116, S5_TX1116, VBUS1116, VDDA_3V1101, VDD_3V1101, VDD_5V_BRICK1116, VDD_5V_IN1116, VDD_SERVO1116: footprint PX4FMUv2.4:PIXHAWK2_PAD.04X.04 -> PIXHAWK2_PAD.04X.04
- JP1, JP2: footprint PX4FMUv2.4:PIXHAWK2_FIDUCIAL-1.5X3 -> PIXHAWK2_FIDUCIAL-1.5X3
- M3_MOUNT1101, M3_MOUNT1102, M3_MOUNT1103, M3_MOUNT1104: footprint PX4FMUv2.4:PIXHAWK2_MOUNT-HOLE3.1 -> PIXHAWK2_MOUNT-HOLE3.1
- OSHW_LOGO1116: footprint PX4FMUv2.4:PIXHAWK2_OSHW-LOGO-S -> PIXHAWK2_OSHW-LOGO-S
- VP_0, VP_1, VP_2, VP_3, VP_33, VP_34, VP_35, VP_41, VP_42, VP_43, VP_51, VP_52, VP_53, VP_54, VP_55, VP_56, VP_57, VP_58, VP_59, VP_60, VP_61: footprint PX4FMUv2.4:VPAD_VPAC0 -> VPAD_VPAC0
- VP_10, VP_11, VP_12, VP_13, VP_14, VP_15, VP_16, VP_17, VP_18, VP_19, VP_20, VP_21, VP_22, VP_23, VP_24, VP_25, VP_26, VP_27, VP_28, VP_29, VP_30, VP_31, VP_32, VP_36, VP_37, VP_39, VP_4, VP_40, VP_44, VP_45, VP_46, VP_47, VP_48, VP_49, VP_5, VP_50, VP_6, VP_7, VP_8, VP_9: footprint PX4FMUv2.4:VPAD_VPAC1 -> VPAD_VPAC1
- VP_38: footprint PX4FMUv2.4:VPAD_VPAC2 -> VPAD_VPAC2
