File: examples/PIXHAWK/kicad_files/PX4FMUv2.4_SS_2.sch (KiCad schematic (older format))
At the start: 30 parts, among them J201 DF13C-6P-1.25V, J202 DF13C-6P-1.25V, J203 DF13C-6P-1.25V, J204 DF13C-6P-1.25V, U201 TXS0108QFN20, U202 TXS0108QFN20

Commit message: force golbale netnames on, to get around fill/net problem
Parts:
- C201, C202: footprint PX4FMUv2.4:PIXHAWK2_0402-CAP -> PIXHAWK2_0402-CAP
- D201, D202, D203: footprint PX4FMUv2.4:PIXHAWK2_0402-TVS -> PIXHAWK2_0402-TVS; Field5 TVS -> (none)
- J201, J202, J203, J204: footprint PX4FMUv2.4:CON-HIROSE-DF13_DF13C-6P-1.25V -> CON-HIROSE-DF13_DF13C-6P-1.25V
- L201, L202, L203: footprint PX4FMUv2.4:PIXHAWK2_KYOCERA-KNH16-DA -> PIXHAWK2_KYOCERA-KNH16-DA
- R201, R202, R203, R204, R205, R206, R207, R208, R209, R210, R211, R212, R213, R214, R215, R216: footprint PX4FMUv2.4:PIXHAWK2_0402-RES -> PIXHAWK2_0402-RES
- U201, U202: footprint PX4FMUv2.4:PIXHAWK2_QFN20-RGY -> PIXHAWK2_QFN20-RGY
Connections:
- wire segments 136 -> 155
