File: examples/PIXHAWK/kicad_files/PX4FMUv2.4_SS_3.sch (KiCad schematic (older format))
At the start: 12 parts, among them J301 47346-0001, J302 DF13C-4P-1.25V, U301 2908-05WB-MG, U302 NUF2042XV6

Commit message: force golbale netnames on, to get around fill/net problem
Parts:
- J301: footprint PX4FMUv2.4:PIXHAWK2_MOLEX-47346-0001 -> PIXHAWK2_MOLEX-47346-0001
- J302: footprint PX4FMUv2.4:CON-HIROSE-DF13_DF13C-4P-1.25V -> CON-HIROSE-DF13_DF13C-4P-1.25V
- JX301: footprint PX4FMUv2.4:PIXHAWK2_FTSH-105-01-XXX-DV-K -> PIXHAWK2_FTSH-105-01-XXX-DV-K
- R301, R302, R303, R304, R305, R306, R307: footprint PX4FMUv2.4:PIXHAWK2_0402-RES -> PIXHAWK2_0402-RES
- U301: footprint PX4FMUv2.4:BASEBOARD_MICROSD -> BASEBOARD_MICROSD
- U302: footprint PX4FMUv2.4:PIXHAWK2_SOT563-6 -> PIXHAWK2_SOT563-6
Connections:
- wire segments 50 -> 71
