File: examples/PIXHAWK/kicad_files/PX4FMUv2.4_SS_4.sch (KiCad schematic (older format))
At the start: 25 parts, among them J401 DF13C-4P-1.25V, J402 DF13C-3P-1.25V, J403 DF13C-7P-1.25V, J404 DF13C-5P-1.25V, J405 DF13C-4P-1.25V, U401 MAX3051

Commit message: force golbale netnames on, to get around fill/net problem
Parts:
- C401, C402: footprint PX4FMUv2.4:PIXHAWK2_0402-CAP -> PIXHAWK2_0402-CAP
- D401, D402, D403, D404: footprint PX4FMUv2.4:PIXHAWK2_0402-TVS -> PIXHAWK2_0402-TVS; Field5 TVS -> (none)
- J401, J405: footprint PX4FMUv2.4:CON-HIROSE-DF13_DF13C-4P-1.25V -> CON-HIROSE-DF13_DF13C-4P-1.25V
- J402: footprint PX4FMUv2.4:CON-HIROSE-DF13_DF13C-3P-1.25V -> CON-HIROSE-DF13_DF13C-3P-1.25V
- J403: footprint PX4FMUv2.4:CON-HIROSE-DF13_DF13C-7P-1.25V -> CON-HIROSE-DF13_DF13C-7P-1.25V
- J404: footprint PX4FMUv2.4:CON-HIROSE-DF13_DF13C-5P-1.25V -> CON-HIROSE-DF13_DF13C-5P-1.25V
- L401, L402, L403, L404: footprint PX4FMUv2.4:PIXHAWK2_KYOCERA-KNH16-DA -> PIXHAWK2_KYOCERA-KNH16-DA
- R401, R402, R403, R404, R405, R406, R407, R408, R409: footprint PX4FMUv2.4:PIXHAWK2_0402-RES -> PIXHAWK2_0402-RES
- U401: footprint PX4FMUv2.4:PIXHAWK2_SOT23-8 -> PIXHAWK2_SOT23-8
Connections:
- wire segments 86 -> 116
