File: examples/PIXHAWK/kicad_files/PX4FMUv2.4_SS_5.sch (KiCad schematic (older format))
At the start: 21 parts, among them U501 L3GD20, U502 L3GD20H, U504 LSM303D, U505 MPU-6000, U506 MS5611-01BA, X503 0512811094

Commit message: force golbale netnames on, to get around fill/net problem
Parts:
- C501, C506, C509, C511: footprint PX4FMUv2.4:PIXHAWK2_0805-CAP -> PIXHAWK2_0805-CAP
- C502, C503, C504, C505, C507, C508, C510, C514: footprint PX4FMUv2.4:PIXHAWK2_0402-CAP -> PIXHAWK2_0402-CAP
- C512, C513, C515: footprint PX4FMUv2.4:PIXHAWK2_0603-CAP -> PIXHAWK2_0603-CAP
- U501: footprint PX4FMUv2.4:PIXHAWK2_L3G4200DH-MAN -> PIXHAWK2_L3G4200DH-MAN
- U502, U504: footprint PX4FMUv2.4:PIXHAWK2_LGA-16L -> PIXHAWK2_LGA-16L
- U505: footprint PX4FMUv2.4:PIXHAWK2_QFN-24 -> PIXHAWK2_QFN-24
- U506: footprint PX4FMUv2.4:PIXHAWK2_MS5611-01BA -> PIXHAWK2_MS5611-01BA
- X503: footprint PX4FMUv2.4:PIXHAWK2_51281-1094 -> PIXHAWK2_51281-1094
Connections:
- wire segments 112 -> 138
