File: examples/PIXHAWK/kicad_files/PX4FMUv2.4_SS_6.sch (KiCad schematic (older format))
At the start: 40 parts, among them Q601 MMBT3906LT1SMD, U101 STM32F4X7VX, U601 BQ24315, U602 BQ24315, U603 MIC5332

Commit message: force golbale netnames on, to get around fill/net problem
Parts:
- B601: footprint PX4FMUv2.4:PIXHAWK2_MS621FE -> PIXHAWK2_MS621FE; Field4 - -> (none)
- C601, C604, C605: footprint PX4FMUv2.4:PIXHAWK2_0805-CAP -> PIXHAWK2_0805-CAP
- C602, C606, C607, C608, C609, C610, C612, C615, C616, C617: footprint PX4FMUv2.4:PIXHAWK2_0402-CAP -> PIXHAWK2_0402-CAP
- C603, C611, C613: footprint PX4FMUv2.4:PIXHAWK2_0603-CAP -> PIXHAWK2_0603-CAP
- C614, C618: footprint PX4FMUv2.4:PIXHAWK2_1206-CAP -> PIXHAWK2_1206-CAP
- D2: footprint PX4FMUv2.4:PIXHAWK2_SOD323 -> PIXHAWK2_SOD323
- L603: footprint PX4FMUv2.4:PIXHAWK2_KYOCERA-KNH16-DA -> PIXHAWK2_KYOCERA-KNH16-DA
- Q601: footprint PX4FMUv2.4:TRANSISTOR-PNP_SOT23-BEC -> TRANSISTOR-PNP_SOT23-BEC
- R602, R603, R604, R608, R609, R610, R611, R615, R616, R617, R620, R635: footprint PX4FMUv2.4:PIXHAWK2_0402-RES -> PIXHAWK2_0402-RES
- R621: footprint PX4FMUv2.4:PIXHAWK2_0603-RES -> PIXHAWK2_0603-RES
- S601: footprint PX4FMUv2.4:PIXHAWK2_EVQP7J01K -> PIXHAWK2_EVQP7J01K
- U101: footprint PX4FMUv2.4:PIXHAWK2_TQFP100 -> PIXHAWK2_TQFP100
- U601, U602: footprint PX4FMUv2.4:PIXHAWK2_QFN8-DSG -> PIXHAWK2_QFN8-DSG
- U603: footprint PX4FMUv2.4:PIXHAWK2_MLF-8-EPAD -> PIXHAWK2_MLF-8-EPAD
Connections:
- wire segments 120 -> 160
