File: examples/PIXHAWK/kicad_files/PX4FMUv2.4_SS_7.sch (KiCad schematic (older format))
At the start: 31 parts, among them J701 DF13C-2P-1.25V, J702 DF13C-3P-1.25V, U701 TCA62724FMG, U702 LT3469, U703 LRTB GFTG-T7AW-1+V7A7-29+R5T9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

Commit message: force golbale netnames on, to get around fill/net problem
Parts:
- C701, C703, C704: footprint PX4FMUv2.4:PIXHAWK2_0402-CAP -> PIXHAWK2_0402-CAP
- C702: footprint PX4FMUv2.4:PIXHAWK2_0603-CAP -> PIXHAWK2_0603-CAP
- D701: footprint PX4FMUv2.4:PIXHAWK2_0402-TVS -> PIXHAWK2_0402-TVS; Field5 TVS -> (none)
- J701: footprint PX4FMUv2.4:CON-HIROSE-DF13_DF13C-2P-1.25V -> CON-HIROSE-DF13_DF13C-2P-1.25V
- J702: footprint PX4FMUv2.4:CON-HIROSE-DF13_DF13C-3P-1.25V -> CON-HIROSE-DF13_DF13C-3P-1.25V
- L701: footprint PX4FMUv2.4:PIXHAWK2_0805-IND -> PIXHAWK2_0805-IND
- LED701, LED702, LED703, LED704, LED705: footprint PX4FMUv2.4:PIXHAWK2_0603-LED -> PIXHAWK2_0603-LED
- R3, R4, R701, R702, R703, R704, R705, R706, R707, R708, R709, R710, R711, R712, R713: footprint PX4FMUv2.4:PIXHAWK2_0402-RES -> PIXHAWK2_0402-RES
- U701: footprint PX4FMUv2.4:PIXHAWK2_SON10 -> PIXHAWK2_SON10; Field4 TCA62724 -> (none)
- U702: footprint PX4FMUv2.4:PIXHAWK2_SOT23-8 -> PIXHAWK2_SOT23-8
- U703: footprint PX4FMUv2.4:PIXHAWK2_6-PLCC -> PIXHAWK2_6-PLCC
Connections:
- wire segments 92 -> 111
