File: examples/PIXHAWK/kicad_files/PX4FMUv2.4_SS_8.sch (KiCad schematic (older format))
At the start: 17 parts, among them J801 JST-ZH-3, U801 STM32F10XCXT6, X801 3.2x2.5 mm / 24 MHz / 15 ppm

Commit message: force golbale netnames on, to get around fill/net problem
Parts:
- C801, C802, C803, C804, C805, C806: footprint PX4FMUv2.4:PIXHAWK2_0402-CAP -> PIXHAWK2_0402-CAP
- D801: footprint PX4FMUv2.4:PIXHAWK2_0402-TVS -> PIXHAWK2_0402-TVS; Field5 TVS -> (none)
- J801: footprint PX4FMUv2.4:FOR-TRANSFERS_JST-ZH-SMT-VERTICAL -> FOR-TRANSFERS_JST-ZH-SMT-VERTICAL
- JX801: footprint PX4FMUv2.4:PIXHAWK2_HEADER_3X01_SMD_H_BOARD_EDGE_SHORT -> PIXHAWK2_HEADER_3X01_SMD_H_BOARD_EDGE_SHORT
- JX802: footprint PX4FMUv2.4:PIXHAWK2_FTSH-105-01-XXX-DV-K -> PIXHAWK2_FTSH-105-01-XXX-DV-K
- R801, R802, R803, R804: footprint PX4FMUv2.4:PIXHAWK2_0402-RES -> PIXHAWK2_0402-RES
- S801: footprint PX4FMUv2.4:PIXHAWK2_EVQP7J01K -> PIXHAWK2_EVQP7J01K
- U801: footprint PX4FMUv2.4:PIXHAWK2_TQFP48 -> PIXHAWK2_TQFP48
- X801: footprint PX4FMUv2.4:PIXHAWK2_OSCILLATOR-3.2X2.5 -> PIXHAWK2_OSCILLATOR-3.2X2.5
Connections:
- wire segments 94 -> 110
