File: examples/PIXHAWK/kicad_files/PX4FMUv2.4_SS_9.sch (KiCad schematic (older format))
At the start: 32 parts, among them U901 TXS0108QFN20, U902 TXS0108QFN20, U903 74LVC2G240

Commit message: force golbale netnames on, to get around fill/net problem
Parts:
- C901, C902, C903: footprint PX4FMUv2.4:PIXHAWK2_0402-CAP -> PIXHAWK2_0402-CAP
- D1: footprint PX4FMUv2.4:PIXHAWK2_MICROSMP -> PIXHAWK2_MICROSMP
- D901, D902, D903: footprint PX4FMUv2.4:PIXHAWK2_0402-TVS -> PIXHAWK2_0402-TVS; Field5 TVS -> (none)
- J901: value ~ -> (none); footprint PX4FMUv2.4:PIXHAWK2_3X16RA -> PIXHAWK2_3X16RA
- L901: footprint PX4FMUv2.4:PIXHAWK2_KYOCERA-KNH16-DA -> PIXHAWK2_KYOCERA-KNH16-DA
- R901, R902, R903, R904, R905, R906, R907, R908, R909, R910, R911, R912, R913, R914, R915, R916, R917, R918, R919, R922: footprint PX4FMUv2.4:PIXHAWK2_0402-RES -> PIXHAWK2_0402-RES
- U901, U902: footprint PX4FMUv2.4:PIXHAWK2_QFN20-RGY -> PIXHAWK2_QFN20-RGY
- U903: footprint PX4FMUv2.4:PIXHAWK2_TSSOP8_SOT505-2 -> PIXHAWK2_TSSOP8_SOT505-2
Connections:
- wire segments 130 -> 151
