File: examples/PIXHAWK/kicad_files/modified_eagle_files/PX4FMUv2.4.brd (EAGLE design)
At the start: 70 x 40.5 mm, 354 parts, among them J201 DF13C-6P-1.25V, J202 DF13C-6P-1.25V, J203 DF13C-6P-1.25V, J204 DF13C-6P-1.25V, J301 47346-0001, J302 DF13C-4P-1.25V, J401 DF13C-4P-1.25V, J402 DF13C-3P-1.25V, J403 DF13C-7P-1.25V, J404 DF13C-5P-1.25V, J405 DF13C-4P-1.25V, J601 DF13C-6P-1.25V, J701 DF13C-2P-1.25V, J702 DF13C-3P-1.25V, J801 JST-ZH-3, M3_MOUNT1101 MOUNT-HOLE3.1MM, M3_MOUNT1102 MOUNT-HOLE3.1MM, M3_MOUNT1103 MOUNT-HOLE3.1MM, M3_MOUNT1104 MOUNT-HOLE3.1MM, Q601 MMBT3906LT1SMD, U1001 BQ24313, U1002 MIC5332, U101 STM32F4X7VX, U102 FM25V01, U1101 LTC4417, U1102 NTHD4102PT1G, U1103 NTHD4102PT1G, U1104 NTHD4102PT1G, U201 TXS0108QFN20, U202 TXS0108QFN20, U301 2908-05WB-MG, U302 NUF2042XV6, U401 MAX3051, U501 L3GD20, U502 L3GD20H, U504 LSM303D, U505 MPU-6000, U506 MS5611-01BA, U601 BQ24315, U602 BQ24315, U603 MIC5332, U701 TCA62724FMG, U702 LT3469, U703 LRTB GFTG-T7AW-1+V7A7-29+R5T9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, U801 STM32F10XCXT6, U901 TXS0108QFN20, U902 TXS0108QFN20, U903 74LVC2G240, X101 3.2x2.5 mm / 24 MHz / 15 ppm, X503 0512811094, X801 3.2x2.5 mm / 24 MHz / 15 ppm

Commit message: blind via which can't be converted to paid, docment with "X" and netname, and via number
Other:
- board text added: "GND:1"
- board text added: "GND:10"
- board text added: "GND:11"
- board text added: "GND:12"
- board text added: "GND:13"
- board text added: "GND:14"
- board text added: "GND:15"
- board text added: "GND:16"
- board text added: "GND:17"
- board text added: "GND:18"
- board text added: "GND:19"
- board text added: "GND:2"
- board text added: "GND:20"
- board text added: "GND:21"
- board text added: "GND:22"
- board text added: "GND:23"
- board text added: "GND:24"
- board text added: "GND:25"
- board text added: "GND:26"
- board text added: "GND:27"
- board text added: "GND:28"
- board text added: "GND:29"
- board text added: "GND:3"
- board text added: "GND:30"
- board text added: "GND:31"
- board text added: "GND:4"
- board text added: "GND:5"
- board text added: "GND:6"
- board text added: "GND:7"
- board text added: "GND:8"
- board text added: "GND:9"
- board text added: "IO-VDD_3V3:32"
- board text added: "IO-VDD_3V3:33"
- board text added: "VBUS:34"
- board text added: "VBUS:35"
- board text added: "VBUS:36"
- board text added: "VDD_3V3_SENSORS:37"
- board text added: "VDD_3V3_SENSORS:38"
- board text added: "VDD_5V_BRICK:39"
- board text added: "VDD_5V_BRICK:40"
- board text added: "VDD_5V_BRICK:41"
- board text added: "VDD_5V_IN:42"
- board text added: "VDD_5V_IN:43"
- board text added: "VDD_5V_IN:44"
- board text added: "VDD_5V_IN:45"
- board text added: "VDD_5V_IN:46"
- board text added: "VDD_5V_IN:47"
- board text added: "VDD_5V_IN:48"
- board text added: "VDD_5V_IN:49"
- board text added: "VDD_5V_IN:50"
- board text added: "VDD_5V_IN:51"
- board text added: "VDD_5V_IN:52"
- board text added: "VDD_5V_IN:53"
- board text added: "VDD_5V_IN:54"
- board text added: "VDD_5V_PERIPH:55"
- board text added: "VDD_5V_PERIPH:56"
- board text added: "VDD_5V_PERIPH:57"
- board text added: "VDD_5V_PERIPH:58"
- board text added: "VDD_5V_PERIPH:59"
- board text added: "VDD_SERVO:60"
- board text added: "VDD_SERVO:61"
- board text added: "VDD_SERVO:62"
- board text removed: "GND"
- board text removed: "IO-VDD_3V3"
- board text removed: "VBUS"
- board text removed: "VDD_3V3_SENSORS"
- board text removed: "VDD_5V_BRICK"
- board text removed: "VDD_5V_IN"
- board text removed: "VDD_5V_PERIPH"
- board text removed: "VDD_SERVO"
